Commit message: Add sensors and update robot model

File: urdf/simple_robot.urdf (robot description, URDF)
Before this commit: robot simple_mobile_robot, 5 links, 4 joints
Links:
- removed link camera_link
- added link caster_wheel; visual sphere radius=0.03
- added link depth_camera_link; visual box size=0.05 0.05 0.03
- added link imu_link; visual box size=0.06 0.06 0.04
Joints:
- removed joint camera_joint
- added joint caster_wheel_joint: type fixed, parent base_link, child caster_wheel, origin xyz=-0.15 0 -0.08 rpy=0 0 0
- added joint depth_camera_joint: type fixed, parent base_link, child depth_camera_link, origin xyz=0.15 0 0.08 rpy=0 0 0
- added joint imu_joint: type fixed, parent base_link, child imu_link, origin xyz=-0.10 0 0.06 rpy=0 0 0
