Commit message: Add Xacro support and Gazebo simulation

File: urdf/simple_robot.urdf.xacro (robot description, xacro)
@@ -36,4 +36,9 @@
       izz="0.1"/>
   </inertial>
+   <collision>
+    <geometry>
+     <box size="${base_length} ${base_width} ${base_height}"/>
+    </geometry>
+  </collision>
  </link>
  <link name="left_wheel">
@@ -57,4 +62,9 @@
       izz="0.001"/>
   </inertial>
+  <collision>
+   <geometry>
+    <cylinder radius="${wheel_radius}" length="${wheel_width}"/>
+   </geometry>
+  </collision>
  </link>
  <joint name="left_wheel_joint" type="continuous">
@@ -84,4 +94,9 @@
       izz="0.001"/>
   </inertial>
+  <collision>
+   <geometry>
+    <cylinder radius="${wheel_radius}" length="${wheel_width}"/>
+   </geometry>
+  </collision>
  </link>
  <joint name="right_wheel_joint" type="continuous">
@@ -102,4 +117,5 @@
   <inertial>
    <mass value="0.2"/>
+   <origin xyz="0 0 0"/>
    <inertia
       ixx="0.0001"
@@ -110,4 +126,9 @@
       izz="0.0001"/>
   </inertial>
+  <collision>
+   <geometry>
+    <cylinder radius="${lidar_radius}" length="${lidar_height}"/>
+   </geometry>
+  </collision>
  </link>
  <joint name="lidar_joint" type="fixed">
@@ -127,4 +148,5 @@
   <inertial>
    <mass value="0.1"/>
+   <origin xyz="0 0 0"/>
    <inertia
       ixx="0.0001"
@@ -135,4 +157,9 @@
       izz="0.0001"/>
   </inertial>
+  <collision>
+   <geometry>
+    <box size="${camera_size_x} ${camera_size_y} ${camera_size_z}"/>
+   </geometry>
+  </collision>
  </link>
  <joint name="depth_camera_joint" type="fixed">
@@ -152,4 +179,5 @@
   <inertial>
    <mass value="0.05"/>
+   <origin xyz="0 0 0"/>
    <inertia
       ixx="0.00001"
@@ -160,4 +188,9 @@
       izz="0.00001"/>
   </inertial>
+  <collision>
+   <geometry>
+    <box size="${imu_size_x} ${imu_size_y} ${imu_size_z}"/>
+   </geometry>
+  </collision>
  </link>
  <joint name="imu_joint" type="fixed">
@@ -177,4 +210,5 @@
   <inertial>
    <mass value="0.2"/>
+   <origin xyz="0 0 0"/>
    <inertia
       ixx="0.0001"
@@ -185,4 +219,9 @@
       izz="0.0001"/>
   </inertial>
+  <collision>
+   <geometry>
+    <sphere radius="${caster_radius}"/>
+   </geometry>
+  </collision>
  </link>
  <joint name="caster_wheel_joint" type="fixed">

Commit message: Add Gazebo launch file for robot simulation

File: urdf/simple_robot.urdf.xacro (robot description, xacro)
@@ -230,3 +230,42 @@
   <origin xyz="-0.15 0 -0.07" rpy="0 0 0"/>
  </joint>
+ <!--adding ros2 control -->
+ <ros2_control name="GazeboSimSystem" type="system">
+  <hardware>
+   <plugin>gz_ros2_control/GazeboSimSystem</plugin>
+  <!--A plugin is like a software module that adds functionality.
+  #Gazebo doesn't automatically understand ROS motor commands.
+  #The plugin acts as a translator.
+  #ROS -> plugin -> Gazebo -->
+  </hardware>
+  <joint name="left_wheel_joint">
+   <command_interface name="velocity">
+    <param name="min">-1</param>
+    <param name="max">1</param>
+   </command_interface>  <!--command  tell ros to control joint by giving velocity speed-->
+   <state_interface name="position"/>  <!--feedback , it tell ros that u can read current position of joint-->
+   <state_interface name="velocity"/>  <!--feedback = reading the current wheel speed-->
+  </joint>
+  <joint name="right_wheel_joint">
+   <command_interface name="velocity">
+    <param name="min">-1</param>
+    <param name="max">1</param>
+   </command_interface>
+   <state_interface name="position"/>
+   <state_interface name="velocity"/>
+  </joint>
+ </ros2_control>
+ <!--adding the Gazebo plugin -->
+ <gazebo>
+  <plugin
+      filename="gz_ros2_control-system"
+      name="gz_ros2_control::GazeboSimROS2ControlPlugin">
+    <ros>
+      <namespace></namespace>
+    </ros>
+    <parameters>
+      /media/zbook/New Volume/ros2_ws/install/simple_mobile_robot/share/simple_mobile_robot/config/controllers.yaml
+    </parameters>
+   </plugin>
+ </gazebo>
 </robot>

Commit message: Add LiDAR, IMU, depth camera and Gazebo sensor world

File: urdf/simple_robot.urdf.xacro (robot description, xacro)
@@ -170,27 +170,27 @@
  <link name="imu_link">
   <visual>
-   <geometry>
-    <box size="${imu_size_x} ${imu_size_y} ${imu_size_z}"/>
-   </geometry>
-   <material name="yellow">
-    <color rgba="1 1 0 1"/>
-   </material>
-  </visual>
-  <inertial>
-   <mass value="0.05"/>
-   <origin xyz="0 0 0"/>
-   <inertia
-      ixx="0.00001"
-      ixy="0"
-      ixz="0"
-      iyy="0.00001"
-      iyz="0"
-      izz="0.00001"/>
-  </inertial>
-  <collision>
-   <geometry>
-    <box size="${imu_size_x} ${imu_size_y} ${imu_size_z}"/>
-   </geometry>
-  </collision>
+    <geometry>
+      <box size="${imu_size_x} ${imu_size_y} ${imu_size_z}"/>
+    </geometry>
+    <material name="yellow">
+      <color rgba="1 1 0 1"/>
+    </material>
+  </visual>
+  <collision>
+    <geometry>
+      <box size="${imu_size_x} ${imu_size_y} ${imu_size_z}"/>
+    </geometry>
+  </collision>
+  <inertial>
+    <mass value="0.1"/>
+    <origin xyz="0 0 0"/>
+    <inertia
+      ixx="0.000166667"
+      ixy="0"
+      ixz="0"
+      iyy="0.000166667"
+      iyz="0"
+      izz="0.000166667"/>
+  </inertial>
  </link>
  <joint name="imu_joint" type="fixed">
@@ -265,7 +265,60 @@
     </ros>
     <parameters>
-      /media/zbook/New Volume/ros2_ws/install/simple_mobile_robot/share/simple_mobile_robot/config/controllers.yaml
+      /media/zbook/Data/ros2_ws/install/simple_mobile_robot/share/simple_mobile_robot/config/controllers.yaml
     </parameters>
    </plugin>
  </gazebo>
+<gazebo reference="lidar_link">
+  <sensor name="lidar_sensor" type="gpu_lidar">
+    <always_on>true</always_on>
+    <update_rate>10</update_rate>
+    <visualize>true</visualize>
+    <topic>scan</topic>
+    <gz_frame_id>lidar_link</gz_frame_id>
+    <lidar>
+      <scan>
+        <horizontal>
+          <samples>720</samples>
+          <resolution>1</resolution>
+          <min_angle>-3.14159</min_angle>
+          <max_angle>3.14159</max_angle>
+        </horizontal>
+      </scan>
+      <range>
+        <min>0.10</min>
+        <max>10.0</max>
+        <resolution>0.01</resolution>
+      </range>
+    </lidar>
+  </sensor>
+</gazebo>
+<gazebo reference="base_link">
+  <sensor name="imu" type="imu">
+    <always_on>true</always_on>
+    <update_rate>100</update_rate>
+    <visualize>true</visualize>
+    <topic>/imu</topic>
+    <enable_metrics>true</enable_metrics>
+  </sensor>
+</gazebo>
+<gazebo reference="depth_camera_link">
+  <sensor name="depth_camera" type="depth_camera">
+    <always_on>true</always_on>
+    <update_rate>30</update_rate>
+    <visualize>true</visualize>
+    <topic>camera</topic>
+    <camera>
+      <horizontal_fov>1.047</horizontal_fov>
+      <image>
+        <width>640</width>
+        <height>480</height>
+        <format>R8G8B8</format>
+      </image>
+      <clip>
+        <near>0.1</near>
+        <far>10.0</far>
+      </clip>
+    </camera>
+  </sensor>
+</gazebo>
 </robot>
